Commit message: fixed the motion of urdf

File: description/gazebo_control.xacro (robot description, xacro)
@@ -9,5 +9,5 @@
             <wheel_diameter>0.07</wheel_diameter>
             <!-- Limits -->
-            <max_wheel_torque>200</max_wheel_torque>
+            <max_wheel_torque>100</max_wheel_torque>
             <max_wheel_acceleration>10.0</max_wheel_acceleration>
             <!-- Output -->

File: description/robot_core.xacro (robot description, xacro)
@@ -27,9 +27,7 @@
             </geometry>
         </collision>
-        <inertial>
-            <origin xyz="0.00029534576286610104 0.0022322897250936216 0.05452869239467857" rpy="0 0 0"/>
-            <mass value="2.0"/>
-            <inertia ixx="0.17336" iyy="0.361758" izz="0.501427" ixy="-0.0" iyz="0.0" ixz="0.003732"/>
-        </inertial>
+        <xacro:inertial_box mass="1.0" x="0.24" y="0.18" z="0.04">
+            <origin xyz="0 0 0" rpy="0 0 0"/>
+        </xacro:inertial_box>
     </link>
     <gazebo reference="chassis">
@@ -57,9 +55,7 @@
             </geometry>
         </collision>
-        <inertial>
-            <origin xyz="0.07723228972509345 0.09776728972509362 -0.0050000000000000044" rpy="0 0 0"/>
-            <mass value="0.2"/>
-            <inertia ixx="0.000205" iyy="0.00037" izz="0.000205" ixy="-0.0" iyz="0.0" ixz="0.0"/>
-        </inertial>
+        <xacro:inertial_cylinder mass="0.2" radius="0.07" length="0.02">
+            <origin xyz="-0.07276771027490646 0.10223271027490656 -0.0050000000000000044" rpy="0 0 0"/>
+        </xacro:inertial_cylinder>
     </link>
     <gazebo reference="left_wheel">
@@ -87,9 +83,7 @@
             </geometry>
         </collision>
-        <inertial>
+        <xacro:inertial_cylinder mass="0.2" radius="0.07" length="0.02">
             <origin xyz="-0.07276771027490646 -0.10223271027490656 -0.0050000000000000044" rpy="0 0 0"/>
-            <mass value="0.2"/>
-            <inertia ixx="0.000205" iyy="0.00037" izz="0.000205" ixy="-0.0" iyz="0.0" ixz="-0.0"/>
-        </inertial>
+        </xacro:inertial_cylinder>
     </link>
     <gazebo reference="right_wheel">
@@ -105,16 +99,16 @@
         <visual>
             <geometry>
-                <sphere radius="0.015" />
-            </geometry>
-            <material name="red">
-                <color rgba="1 0 0 1"/>
-            </material>
-        </visual>
-        <collision>
-            <geometry>
-                <sphere radius="0.015" />
-            </geometry>
-        </collision>
-        <xacro:inertial_sphere mass="0.1" radius="0.015">
+                <sphere radius="0.014" />
+            </geometry>
+            <material name="red">
+                <color rgba="1 0 0 1"/>
+            </material>
+        </visual>
+        <collision>
+            <geometry>
+                <sphere radius="0.014" />
+            </geometry>
+        </collision>
+        <xacro:inertial_sphere mass="0.1" radius="0.014">
             <origin xyz="0 0 0" rpy="0 0 0"/>
         </xacro:inertial_sphere>
@@ -122,4 +116,6 @@
     <gazebo reference="front_caster_wheel_one">
         <material>Gazebo/Black</material>
+        <mu1>0.005</mu1>
+        <mu2>0.005</mu2>
     </gazebo>
     <!-- FRONT CASTER WHEEL 2 LINK -->
@@ -132,16 +128,16 @@
         <visual>
             <geometry>
-                <sphere radius="0.015" />
-            </geometry>
-            <material name="red">
-                <color rgba="1 0 0 1"/>
-            </material>
-        </visual>
-        <collision>
-            <geometry>
-                <sphere radius="0.015" />
-            </geometry>
-        </collision>
-        <xacro:inertial_sphere mass="0.1" radius="0.015">
+                <sphere radius="0.014" />
+            </geometry>
+            <material name="red">
+                <color rgba="1 0 0 1"/>
+            </material>
+        </visual>
+        <collision>
+            <geometry>
+                <sphere radius="0.014" />
+            </geometry>
+        </collision>
+        <xacro:inertial_sphere mass="0.1" radius="0.014">
             <origin xyz="0 0 0" rpy="0 0 0"/>
         </xacro:inertial_sphere>
@@ -149,4 +145,6 @@
     <gazebo reference="front_caster_wheel_two">
         <material>Gazebo/Black</material>
+        <mu1>0.005</mu1>
+        <mu2>0.005</mu2>
     </gazebo>
     <!-- Back CASTER WHEEL 1 LINK -->
@@ -159,16 +157,16 @@
         <visual>
             <geometry>
-                <sphere radius="0.015" />
-            </geometry>
-            <material name="red">
-                <color rgba="1 0 0 1"/>
-            </material>
-        </visual>
-        <collision>
-            <geometry>
-                <sphere radius="0.015" />
-            </geometry>
-        </collision>
-        <xacro:inertial_sphere mass="0.1" radius="0.015">
+                <sphere radius="0.014" />
+            </geometry>
+            <material name="red">
+                <color rgba="1 0 0 1"/>
+            </material>
+        </visual>
+        <collision>
+            <geometry>
+                <sphere radius="0.014" />
+            </geometry>
+        </collision>
+        <xacro:inertial_sphere mass="0.1" radius="0.014">
             <origin xyz="0 0 0" rpy="0 0 0"/>
         </xacro:inertial_sphere>
@@ -176,4 +174,6 @@
     <gazebo reference="back_caster_wheel_one">
         <material>Gazebo/Black</material>
+        <mu1>0.005</mu1>
+        <mu2>0.005</mu2>
     </gazebo>
     <!-- Back CASTER WHEEL 2 LINK -->
@@ -186,16 +186,16 @@
         <visual>
             <geometry>
-                <sphere radius="0.015" />
-            </geometry>
-            <material name="red">
-                <color rgba="1 0 0 1"/>
-            </material>
-        </visual>
-        <collision>
-            <geometry>
-                <sphere radius="0.015" />
-            </geometry>
-        </collision>
-        <xacro:inertial_sphere mass="0.1" radius="0.015">
+                <sphere radius="0.014" />
+            </geometry>
+            <material name="red">
+                <color rgba="1 0 0 1"/>
+            </material>
+        </visual>
+        <collision>
+            <geometry>
+                <sphere radius="0.014" />
+            </geometry>
+        </collision>
+        <xacro:inertial_sphere mass="0.1" radius="0.014">
             <origin xyz="0 0 0" rpy="0 0 0"/>
         </xacro:inertial_sphere>
@@ -203,4 +203,6 @@
     <gazebo reference="back_caster_wheel_two">
         <material>Gazebo/Black</material>
+        <mu1>0.005</mu1>
+        <mu2>0.005</mu2>
     </gazebo>
 </robot>
