Commit message: added urdf

File: description/robot.urdf.xacro (robot description, xacro)
@@ -2,3 +2,4 @@
 <robot xmlns:xacro="http://www.ros.org/wiki/xacro"  name="robot">
     <xacro:include filename="$(find articubot_two)/description/robot_core.xacro" />
+    <xacro:include filename="$(find articubot_two)/description/gazebo_control.xacro" />
 </robot>

File: description/robot_core.xacro (robot description, xacro)
@@ -16,21 +16,24 @@
             <origin xyz="0 0 0" rpy="0 0 0"/>
             <geometry>
-                <mesh filename="package://articubot_two/meshes/chassis.stl" scale="0.001 0.001 0.001"/>
+                <mesh filename="file://$(find articubot_two)/meshes/chassis.stl" scale="0.001 0.001 0.001"/>
             </geometry>
             <material name="grey">
-                <color rgba="0.5 0.5 0.5 1"/>x`
-            </material>
-        </visual>
-        <collision>
-            <geometry>
-                <mesh filename="package://articubot_two/meshes/chassis.stl" scale="0.001 0.001 0.001"/>
+                <color rgba="0.5 0.5 0.5 1"/>
+            </material>
+        </visual>
+        <collision>
+            <geometry>
+                <mesh filename="file://$(find articubot_two)/meshes/chassis.stl" scale="0.001 0.001 0.001"/>
             </geometry>
         </collision>
         <inertial>
             <origin xyz="0.00029534576286610104 0.0022322897250936216 0.05452869239467857" rpy="0 0 0"/>
-            <mass value="37.432583629741174"/>
+            <mass value="2.0"/>
             <inertia ixx="0.17336" iyy="0.361758" izz="0.501427" ixy="-0.0" iyz="0.0" ixz="0.003732"/>
         </inertial>
     </link>
+    <gazebo reference="chassis">
+        <material>Gazebo/White</material>
+    </gazebo>
     <!-- LEFT WHEEL LINK -->
     <joint name="left_wheel_joint" type="continuous">
@@ -43,5 +46,5 @@
         <visual>
             <geometry>
-                <mesh filename="package://articubot_two/meshes/wheel.stl" scale="0.001 0.001 0.001"/>
+                <mesh filename="file://$(find articubot_two)/meshes/wheel.stl" scale="0.001 0.001 0.001"/>
             </geometry>
             <material name="blue">
@@ -51,13 +54,16 @@
         <collision>
             <geometry>
-                <mesh filename="package://articubot_two/meshes/wheel.stl" scale="0.001 0.001 0.001"/>
+                <mesh filename="file://$(find articubot_two)/meshes/wheel.stl" scale="0.001 0.001 0.001"/>
             </geometry>
         </collision>
         <inertial>
-    <origin xyz="0.07723228972509345 0.09776728972509362 -0.0050000000000000044" rpy="0 0 0"/>
-    <mass value="0.6042068071016568"/>
-    <inertia ixx="0.000205" iyy="0.00037" izz="0.000205" ixy="-0.0" iyz="0.0" ixz="0.0"/>
-  </inertial>
-    </link>
+            <origin xyz="0.07723228972509345 0.09776728972509362 -0.0050000000000000044" rpy="0 0 0"/>
+            <mass value="0.2"/>
+            <inertia ixx="0.000205" iyy="0.00037" izz="0.000205" ixy="-0.0" iyz="0.0" ixz="0.0"/>
+        </inertial>
+    </link>
+    <gazebo reference="left_wheel">
+        <material>Gazebo/Blue</material>
+    </gazebo>
     <!-- RIGHT WHEEL LINK -->
     <joint name="right_wheel_joint" type="continuous">
@@ -70,5 +76,5 @@
         <visual>
             <geometry>
-                <mesh filename="package://articubot_two/meshes/wheel.stl" scale="0.001 0.001 0.001"/>
+                <mesh filename="file://$(find articubot_two)/meshes/wheel.stl" scale="0.001 0.001 0.001"/>
             </geometry>
             <material name="blue">
@@ -78,60 +84,123 @@
         <collision>
             <geometry>
-                <mesh filename="package://articubot_two/meshes/wheel.stl" scale="0.001 0.001 0.001"/>
+                <mesh filename="file://$(find articubot_two)/meshes/wheel.stl" scale="0.001 0.001 0.001"/>
             </geometry>
         </collision>
         <inertial>
             <origin xyz="-0.07276771027490646 -0.10223271027490656 -0.0050000000000000044" rpy="0 0 0"/>
-            <mass value="0.6042068071016568"/>
+            <mass value="0.2"/>
             <inertia ixx="0.000205" iyy="0.00037" izz="0.000205" ixy="-0.0" iyz="0.0" ixz="-0.0"/>
         </inertial>
     </link>
-    <!-- FRONT CASTER WHEEL LINK -->
-    <joint name="front_caster_wheel_joint" type="fixed">
-        <parent link="chassis"/>
-        <child link="front_caster_wheel"/>
-        <origin xyz="0.12 0 0" rpy="0 0 0"/>
-    </joint>
-    <link name="front_caster_wheel">
-        <visual>
-            <geometry>
-                <sphere radius="0.015" />
-            </geometry>
-            <material name="red">
-                <color rgba="1 0 0 1"/>
-            </material>
-        </visual>
-        <collision>
-            <geometry>
-                <sphere radius="0.015" />
-            </geometry>
-        </collision>
-        <xacro:inertial_sphere mass="0.1" radius="0.015">
-            <origin xyz="0 0 0" rpy="0 0 0"/>
-        </xacro:inertial_sphere>
-    </link>
-    <!-- Back CASTER WHEEL LINK -->
-    <joint name="back_caster_wheel_joint" type="fixed">
-        <parent link="chassis"/>
-        <child link="back_caster_wheel"/>
-        <origin xyz="-0.12 0 0" rpy="0 0 0"/>
-    </joint>
-    <link name="back_caster_wheel">
-        <visual>
-            <geometry>
-                <sphere radius="0.015" />
-            </geometry>
-            <material name="red">
-                <color rgba="1 0 0 1"/>
-            </material>
-        </visual>
-        <collision>
-            <geometry>
-                <sphere radius="0.015" />
-            </geometry>
-        </collision>
-        <xacro:inertial_sphere mass="0.1" radius="0.015">
-            <origin xyz="0 0 0" rpy="0 0 0"/>
-        </xacro:inertial_sphere>
-    </link>
+    <gazebo reference="right_wheel">
+        <material>Gazebo/Blue</material>
+    </gazebo>
+    <!-- FRONT CASTER WHEEL 1 LINK -->
+    <joint name="front_caster_wheel_one_joint" type="fixed">
+        <parent link="chassis"/>
+        <child link="front_caster_wheel_one"/>
+        <origin xyz="0.12 0.09 0" rpy="0 0 0"/>
+    </joint>
+    <link name="front_caster_wheel_one">
+        <visual>
+            <geometry>
+                <sphere radius="0.015" />
+            </geometry>
+            <material name="red">
+                <color rgba="1 0 0 1"/>
+            </material>
+        </visual>
+        <collision>
+            <geometry>
+                <sphere radius="0.015" />
+            </geometry>
+        </collision>
+        <xacro:inertial_sphere mass="0.1" radius="0.015">
+            <origin xyz="0 0 0" rpy="0 0 0"/>
+        </xacro:inertial_sphere>
+    </link>
+    <gazebo reference="front_caster_wheel_one">
+        <material>Gazebo/Black</material>
+    </gazebo>
+    <!-- FRONT CASTER WHEEL 2 LINK -->
+    <joint name="front_caster_wheel_two_joint" type="fixed">
+        <parent link="chassis"/>
+        <child link="front_caster_wheel_two"/>
+        <origin xyz="0.12 -0.09 0" rpy="0 0 0"/>
+    </joint>
+    <link name="front_caster_wheel_two">
+        <visual>
+            <geometry>
+                <sphere radius="0.015" />
+            </geometry>
+            <material name="red">
+                <color rgba="1 0 0 1"/>
+            </material>
+        </visual>
+        <collision>
+            <geometry>
+                <sphere radius="0.015" />
+            </geometry>
+        </collision>
+        <xacro:inertial_sphere mass="0.1" radius="0.015">
+            <origin xyz="0 0 0" rpy="0 0 0"/>
+        </xacro:inertial_sphere>
+    </link>
+    <gazebo reference="front_caster_wheel_two">
+        <material>Gazebo/Black</material>
+    </gazebo>
+    <!-- Back CASTER WHEEL 1 LINK -->
+    <joint name="back_caster_wheel_one_joint" type="fixed">
+        <parent link="chassis"/>
+        <child link="back_caster_wheel_one"/>
+        <origin xyz="-0.12 0.09 0" rpy="0 0 0"/>
+    </joint>
+    <link name="back_caster_wheel_one">
+        <visual>
+            <geometry>
+                <sphere radius="0.015" />
+            </geometry>
+            <material name="red">
+                <color rgba="1 0 0 1"/>
+            </material>
+        </visual>
+        <collision>
+            <geometry>
+                <sphere radius="0.015" />
+            </geometry>
+        </collision>
+        <xacro:inertial_sphere mass="0.1" radius="0.015">
+            <origin xyz="0 0 0" rpy="0 0 0"/>
+        </xacro:inertial_sphere>
+    </link>
+    <gazebo reference="back_caster_wheel_one">
+        <material>Gazebo/Black</material>
+    </gazebo>
+    <!-- Back CASTER WHEEL 2 LINK -->
+    <joint name="back_caster_wheel_two_joint" type="fixed">
+        <parent link="chassis"/>
+        <child link="back_caster_wheel_two"/>
+        <origin xyz="-0.12 -0.09 0" rpy="0 0 0"/>
+    </joint>
+    <link name="back_caster_wheel_two">
+        <visual>
+            <geometry>
+                <sphere radius="0.015" />
+            </geometry>
+            <material name="red">
+                <color rgba="1 0 0 1"/>
+            </material>
+        </visual>
+        <collision>
+            <geometry>
+                <sphere radius="0.015" />
+            </geometry>
+        </collision>
+        <xacro:inertial_sphere mass="0.1" radius="0.015">
+            <origin xyz="0 0 0" rpy="0 0 0"/>
+        </xacro:inertial_sphere>
+    </link>
+    <gazebo reference="back_caster_wheel_two">
+        <material>Gazebo/Black</material>
+    </gazebo>
 </robot>

Commit message: added ekf nd imu for rotation for simulation

File: description/robot.urdf.xacro (robot description, xacro)
@@ -6,3 +6,4 @@
     <xacro:include filename="$(find articubot_two)/description/lidar.xacro" />
     <xacro:include filename="$(find articubot_two)/description/camera.xacro" />
+    <xacro:include filename="$(find articubot_two)/description/imu.xacro" />
 </robot>

File: description/robot_core.xacro (robot description, xacro)
@@ -52,5 +52,5 @@
         <collision>
             <geometry>
-                <mesh filename="file://$(find articubot_two)/meshes/wheel.stl" scale="0.001 0.001 0.001"/>
+                <sphere radius="0.035" />
             </geometry>
         </collision>
@@ -82,5 +82,5 @@
         <collision>
             <geometry>
-                <mesh filename="file://$(find articubot_two)/meshes/wheel.stl" scale="0.001 0.001 0.001"/>
+                <sphere radius="0.035" />
             </geometry>
         </collision>
