Commit message: updated to correct launch_sim

File: description/camera.xacro (robot description, xacro)
@@ -1,4 +1,5 @@
 <?xml version="1.0"?>
-<robot xmlns:xacro="http://www.ros.org/wiki/xacro" >
+<robot xmlns:xacro="http://www.ros.org/wiki/xacro">
+    <!-- CAMERA MOUNT -->
     <joint name="camera_joint" type="fixed">
         <parent link="chassis"/>
@@ -6,12 +7,52 @@
         <origin xyz="0.15 0 0.08" rpy="0 0 0"/>
     </joint>
+    <!-- CAMERA LINK -->
     <link name="camera_link">
+        <!-- VISUAL -->
         <visual>
             <geometry>
-                <box size="0.009 0.03 0.03"/>
+                <box size="0.03 0.03 0.03"/>
             </geometry>
             <material name="red"/>
         </visual>
+        <!-- COLLISION -->
+        <collision>
+            <geometry>
+                <box size="0.03 0.03 0.03"/>
+            </geometry>
+        </collision>
+        <!-- INERTIAL -->
+        <inertial>
+            <origin xyz="0 0 0"/>
+            <mass value="0.1"/>
+            <inertia
+                ixx="0.0001"
+                ixy="0.0"
+                ixz="0.0"
+                iyy="0.0001"
+                iyz="0.0"
+                izz="0.0001"/>
+        </inertial>
+        <!-- CAMERA SENSOR FOR GAZEBO HARMONIC -->
+        <sensor name="camera_sensor" type="camera">
+            <always_on>true</always_on>
+            <visualize>true</visualize>
+            <update_rate>30</update_rate>
+            <topic>/camera</topic>
+            <camera>
+                <horizontal_fov>1.047</horizontal_fov>
+                <image>
+                    <width>640</width>
+                    <height>480</height>
+                    <format>R8G8B8</format>
+                </image>
+                <clip>
+                    <near>0.1</near>
+                    <far>100</far>
+                </clip>
+            </camera>
+        </sensor>
     </link>
+    <!-- OPTICAL FRAME -->
     <joint name="camera_optical_joint" type="fixed">
         <parent link="camera_link"/>
@@ -19,27 +60,4 @@
         <origin xyz="0 0 0" rpy="${-pi/2} 0 ${-pi/2}"/>
     </joint>
-    <link name="camera_link_optical"></link>
-    <gazebo reference="camera_link">
-        <material>Gazebo/Red</material>
-        <sensor name="camera" type="camera">
-            <pose> 0 0 0 0 0 0 </pose>
-            <visualize>true</visualize>
-            <update_rate>30</update_rate>
-            <camera>
-                <horizontal_fov>0.933</horizontal_fov>
-                <image>
-                    <format>R8G8B8</format>
-                    <width>640</width>
-                    <height>480</height>
-                </image>
-                <clip>
-                    <near>0.1</near>
-                    <far>100.0</far>
-                </clip>
-            </camera>
-            <plugin name="camera_controller" filename="libgazebo_ros_camera.so">
-                <frame_name>camera_link_optical</frame_name>
-            </plugin>
-        </sensor>
-    </gazebo>
+    <link name="camera_link_optical"/>
 </robot>

File: description/lidar.xacro (robot description, xacro)
@@ -1,36 +1,44 @@
 <?xml version="1.0"?>
-<robot xmlns:xacro="http://www.ros.org/wiki/xacro">
+<robot xmlns:xacro="http://www.ros.org/wiki/xacro" >
     <joint name="laser_joint" type="fixed">
-        <parent link="base_link"/>
+        <parent link="chassis"/>
         <child link="laser_frame"/>
-        <origin xyz="-0.06 0 0.096" rpy="0 0 0"/>
+        <origin xyz="0.122 0 0.212" rpy="0 0 0"/>
     </joint>
     <link name="laser_frame">
         <visual>
             <geometry>
-                <mesh filename="file://$(find articubot_two)/meshes/lidar.stl" scale="0.001 0.001 0.001"/>
+                <cylinder radius="0.05" length="0.04"/>
             </geometry>
-            <material name="red">
-                <color rgba="1 0 0 1"/>
-            </material>
+            <material name="black"/>
+        </visual>
+        <visual>
+            <origin xyz="0 0 -0.05"/>
+            <geometry>
+                <cylinder radius="0.01" length="0.1"/>
+            </geometry>
+            <material name="black"/>
         </visual>
         <collision>
             <geometry>
-                <mesh filename="file://$(find articubot_two)/meshes/lidar.stl" scale="0.001 0.001 0.001"/>
+                <cylinder radius="0.05" length="0.04"/>
             </geometry>
         </collision>
+        <xacro:inertial_cylinder mass="0.1" length="0.04" radius="0.05">
+            <origin xyz="0 0 0" rpy="0 0 0"/>
+        </xacro:inertial_cylinder>
     </link>
     <gazebo reference="laser_frame">
-        <sensor name="laser" type="ray">
-            <pose> 0 0 0 0 0 0 </pose>
-            <visualize>true</visualize>
+        <material>Gazebo/Black</material>
+        <sensor name="laser" type="gpu_lidar">
+            <pose>0 0 0 0 0 0</pose>
+            <visualize>false</visualize>
             <update_rate>10</update_rate>
-            <ray>
+            <topic>scan</topic>
+            <lidar>
                 <scan>
                     <horizontal>
-                        <!-- <samples>180</samples> -->
-                        <!-- <min_angle>-1.57</min_angle> -->
-                        <!-- <max_angle>1.57</max_angle> -->
                         <samples>360</samples>
+                        <resolution>1</resolution>
                         <min_angle>-3.14</min_angle>
                         <max_angle>3.14</max_angle>
@@ -39,16 +47,10 @@
                 <range>
                     <min>0.3</min>
-                    <max>12</max>
+                    <max>12.0</max>
+                    <resolution>0.01</resolution>
                 </range>
-            </ray>
-            <plugin name="laser_controller" filename="libgazebo_ros_ray_sensor.so">
-                <ros>
-                    <argument>~/out:=scan</argument>
-                </ros>
-                <output_type>sensor_msgs/LaserScan</output_type>
-                <frame_name>laser_frame</frame_name>
-            </plugin>
+            </lidar>
+            <always_on>true</always_on>
         </sensor>
-        <material>Gazebo/Red</material>
     </gazebo>
 </robot>

File: description/robot.urdf.xacro (robot description, xacro)
@@ -1,5 +1,4 @@
 <?xml version="1.0"?>
 <robot xmlns:xacro="http://www.ros.org/wiki/xacro"  name="robot">
-    <xacro:arg name="sim_mode" default="false"/>
     <xacro:include filename="$(find articubot_two)/description/robot_core.xacro" />
 </robot>
