Commit message: added urdf

File: description/robot_core.xacro (robot description, xacro)
@@ -1,5 +1,5 @@
 <?xml version="1.0"?>
 <robot xmlns:xacro="http://www.ros.org/wiki/xacro">
-    <xacro:include filename="$(find articubot_two)/description/material_color.xacro" />
+    <!-- TO DO <xacro:include filename="$(find articubot_two)/description/material_color.xacro" /> -->
     <!-- BASE LINK -->
     <link name="base_link">
@@ -17,4 +17,7 @@
                 <mesh filename="package://articubot_two/meshes/chassis.stl" scale="0.001 0.001 0.001"/>
             </geometry>
+            <material name="grey">
+                <color rgba="0.5 0.5 0.5 1"/>
+            </material>
         </visual>
         <collision>
@@ -28,17 +31,83 @@
         <parent link="base_link"/>
         <child link="left_wheel"/>
-        <origin xyz="0 0.0.15 0" rpy="0 0 0"/>
-        <axis xyz="0 1 0"/>
+        <origin xyz="0 0.09 0.02" rpy="${-pi/2} 0 0"/>
+        <axis xyz="0 0 1"/>
     </joint>
     <link name="left_wheel">
         <visual>
-            <origin xyz="0 0 0" rpy="0 0 0"/>
             <geometry>
-                <mesh filename="package://articubot_two/meshes/left_wheel.stl" scale="0.001 0.001 0.001"/>
+                <mesh filename="package://articubot_two/meshes/wheel.stl" scale="0.001 0.001 0.001"/>
             </geometry>
+            <material name="blue">
+                <color rgba="0 0 1 1"/>
+            </material>
         </visual>
         <collision>
             <geometry>
-                <mesh filename="package://articubot_two/meshes/left_wheel.stl" scale="0.001 0.001 0.001"/>
+                <mesh filename="package://articubot_two/meshes/wheel.stl" scale="0.001 0.001 0.001"/>
+            </geometry>
+        </collision>
+    </link>
+    <!-- RIGHT WHEEL LINK -->
+    <joint name="right_wheel_joint" type="continuous">
+        <parent link="base_link"/>
+        <child link="right_wheel"/>
+        <origin xyz="0 -0.09 0.02" rpy="${pi/2} 0 0"/>
+        <axis xyz="0 0 -1"/>
+    </joint>
+    <link name="right_wheel">
+        <visual>
+            <geometry>
+                <mesh filename="package://articubot_two/meshes/wheel.stl" scale="0.001 0.001 0.001"/>
+            </geometry>
+            <material name="blue">
+                <color rgba="0 0 1 1"/>
+            </material>
+        </visual>
+        <collision>
+            <geometry>
+                <mesh filename="package://articubot_two/meshes/wheel.stl" scale="0.001 0.001 0.001"/>
+            </geometry>
+        </collision>
+    </link>
+    <!-- FRONT CASTER WHEEL LINK -->
+    <joint name="front_caster_wheel_joint" type="fixed">
+        <parent link="chassis"/>
+        <child link="front_caster_wheel"/>
+        <origin xyz="0.12 0 0" rpy="0 0 0"/>
+    </joint>
+    <link name="front_caster_wheel">
+        <visual>
+            <geometry>
+                <sphere radius="0.015" />
+            </geometry>
+            <material name="red">
+                <color rgba="1 0 0 1"/>
+            </material>
+        </visual>
+        <collision>
+            <geometry>
+                <sphere radius="0.015" />
+            </geometry>
+        </collision>
+    </link>
+    <!-- Back CASTER WHEEL LINK -->
+    <joint name="back_caster_wheel_joint" type="fixed">
+        <parent link="chassis"/>
+        <child link="back_caster_wheel"/>
+        <origin xyz="-0.12 0 0" rpy="0 0 0"/>
+    </joint>
+    <link name="back_caster_wheel">
+        <visual>
+            <geometry>
+                <sphere radius="0.015" />
+            </geometry>
+            <material name="red">
+                <color rgba="1 0 0 1"/>
+            </material>
+        </visual>
+        <collision>
+            <geometry>
+                <sphere radius="0.015" />
             </geometry>
         </collision>

Commit message: done with the urdf

File: description/robot_core.xacro (robot description, xacro)
@@ -2,4 +2,5 @@
 <robot xmlns:xacro="http://www.ros.org/wiki/xacro">
     <!-- TO DO <xacro:include filename="$(find articubot_two)/description/material_color.xacro" /> -->
+    <xacro:include filename="$(find articubot_two)/description/inertial_macros.xacro" />
     <!-- BASE LINK -->
     <link name="base_link">
@@ -18,5 +19,5 @@
             </geometry>
             <material name="grey">
-                <color rgba="0.5 0.5 0.5 1"/>
+                <color rgba="0.5 0.5 0.5 1"/>x`
             </material>
         </visual>
@@ -26,4 +27,9 @@
             </geometry>
         </collision>
+        <inertial>
+            <origin xyz="0.00029534576286610104 0.0022322897250936216 0.05452869239467857" rpy="0 0 0"/>
+            <mass value="37.432583629741174"/>
+            <inertia ixx="0.17336" iyy="0.361758" izz="0.501427" ixy="-0.0" iyz="0.0" ixz="0.003732"/>
+        </inertial>
     </link>
     <!-- LEFT WHEEL LINK -->
@@ -48,4 +54,9 @@
             </geometry>
         </collision>
+        <inertial>
+    <origin xyz="0.07723228972509345 0.09776728972509362 -0.0050000000000000044" rpy="0 0 0"/>
+    <mass value="0.6042068071016568"/>
+    <inertia ixx="0.000205" iyy="0.00037" izz="0.000205" ixy="-0.0" iyz="0.0" ixz="0.0"/>
+  </inertial>
     </link>
     <!-- RIGHT WHEEL LINK -->
@@ -70,4 +81,9 @@
             </geometry>
         </collision>
+        <inertial>
+            <origin xyz="-0.07276771027490646 -0.10223271027490656 -0.0050000000000000044" rpy="0 0 0"/>
+            <mass value="0.6042068071016568"/>
+            <inertia ixx="0.000205" iyy="0.00037" izz="0.000205" ixy="-0.0" iyz="0.0" ixz="-0.0"/>
+        </inertial>
     </link>
     <!-- FRONT CASTER WHEEL LINK -->
@@ -91,4 +107,7 @@
             </geometry>
         </collision>
+        <xacro:inertial_sphere mass="0.1" radius="0.015">
+            <origin xyz="0 0 0" rpy="0 0 0"/>
+        </xacro:inertial_sphere>
     </link>
     <!-- Back CASTER WHEEL LINK -->
@@ -112,4 +131,7 @@
             </geometry>
         </collision>
+        <xacro:inertial_sphere mass="0.1" radius="0.015">
+            <origin xyz="0 0 0" rpy="0 0 0"/>
+        </xacro:inertial_sphere>
     </link>
 </robot>

Commit message: fixed the wobbling for bot

File: description/robot_core.xacro (robot description, xacro)
@@ -56,9 +56,11 @@
         </collision>
         <xacro:inertial_cylinder mass="0.2" radius="0.07" length="0.02">
-            <origin xyz="-0.07276771027490646 0.10223271027490656 -0.0050000000000000044" rpy="0 0 0"/>
+            <origin xyz="0 0 0" rpy="0 0 0"/>
         </xacro:inertial_cylinder>
     </link>
     <gazebo reference="left_wheel">
         <material>Gazebo/Blue</material>
+        <mu1>1.0</mu1>
+        <mu2>1.0</mu2>
     </gazebo>
     <!-- RIGHT WHEEL LINK -->
@@ -84,20 +86,22 @@
         </collision>
         <xacro:inertial_cylinder mass="0.2" radius="0.07" length="0.02">
-            <origin xyz="-0.07276771027490646 -0.10223271027490656 -0.0050000000000000044" rpy="0 0 0"/>
+            <origin xyz="0 0 0" rpy="0 0 0"/>
         </xacro:inertial_cylinder>
     </link>
     <gazebo reference="right_wheel">
         <material>Gazebo/Blue</material>
+        <mu1>1.0</mu1>
+        <mu2>1.0</mu2>
     </gazebo>
-    <!-- FRONT CASTER WHEEL 1 LINK -->
+    <!-- FRONT CASTER WHEEL LINK -->
     <joint name="front_caster_wheel_one_joint" type="fixed">
         <parent link="chassis"/>
         <child link="front_caster_wheel_one"/>
-        <origin xyz="0.12 0.09 0" rpy="0 0 0"/>
+        <origin xyz="0.12 0 0" rpy="0 0 0"/>
     </joint>
     <link name="front_caster_wheel_one">
         <visual>
             <geometry>
-                <sphere radius="0.014" />
+                <sphere radius="0.01495" />
             </geometry>
             <material name="red">
@@ -107,8 +111,8 @@
         <collision>
             <geometry>
-                <sphere radius="0.014" />
+                <sphere radius="0.01495" />
             </geometry>
         </collision>
-        <xacro:inertial_sphere mass="0.1" radius="0.014">
+        <xacro:inertial_sphere mass="0.1" radius="0.01495">
             <origin xyz="0 0 0" rpy="0 0 0"/>
         </xacro:inertial_sphere>
@@ -116,17 +120,17 @@
     <gazebo reference="front_caster_wheel_one">
         <material>Gazebo/Black</material>
-        <mu1>0.005</mu1>
-        <mu2>0.005</mu2>
+        <mu1>0.0001</mu1>
+        <mu2>0.0001</mu2>
     </gazebo>
-    <!-- FRONT CASTER WHEEL 2 LINK -->
-    <joint name="front_caster_wheel_two_joint" type="fixed">
+    <!-- Back caster wheel -->
+    <joint name="back_caster_wheel_one_joint" type="fixed">
         <parent link="chassis"/>
-        <child link="front_caster_wheel_two"/>
-        <origin xyz="0.12 -0.09 0" rpy="0 0 0"/>
+        <child link="back_caster_wheel_one"/>
+        <origin xyz="-0.12 0 0" rpy="0 0 0"/>
     </joint>
-    <link name="front_caster_wheel_two">
+    <link name="back_caster_wheel_one">
         <visual>
             <geometry>
-                <sphere radius="0.014" />
+                <sphere radius="0.01495" />
             </geometry>
             <material name="red">
@@ -136,37 +140,8 @@
         <collision>
             <geometry>
-                <sphere radius="0.014" />
+                <sphere radius="0.01495" />
             </geometry>
         </collision>
-        <xacro:inertial_sphere mass="0.1" radius="0.014">
-            <origin xyz="0 0 0" rpy="0 0 0"/>
-        </xacro:inertial_sphere>
-    </link>
-    <gazebo reference="front_caster_wheel_two">
-        <material>Gazebo/Black</material>
-        <mu1>0.005</mu1>
-        <mu2>0.005</mu2>
-    </gazebo>
-    <!-- Back CASTER WHEEL 1 LINK -->
-    <joint name="back_caster_wheel_one_joint" type="fixed">
-        <parent link="chassis"/>
-        <child link="back_caster_wheel_one"/>
-        <origin xyz="-0.12 0.09 0" rpy="0 0 0"/>
-    </joint>
-    <link name="back_caster_wheel_one">
-        <visual>
-            <geometry>
-                <sphere radius="0.014" />
-            </geometry>
-            <material name="red">
-                <color rgba="1 0 0 1"/>
-            </material>
-        </visual>
-        <collision>
-            <geometry>
-                <sphere radius="0.014" />
-            </geometry>
-        </collision>
-        <xacro:inertial_sphere mass="0.1" radius="0.014">
+        <xacro:inertial_sphere mass="0.1" radius="0.01495">
             <origin xyz="0 0 0" rpy="0 0 0"/>
         </xacro:inertial_sphere>
@@ -174,35 +149,6 @@
     <gazebo reference="back_caster_wheel_one">
         <material>Gazebo/Black</material>
-        <mu1>0.005</mu1>
-        <mu2>0.005</mu2>
-    </gazebo>
-    <!-- Back CASTER WHEEL 2 LINK -->
-    <joint name="back_caster_wheel_two_joint" type="fixed">
-        <parent link="chassis"/>
-        <child link="back_caster_wheel_two"/>
-        <origin xyz="-0.12 -0.09 0" rpy="0 0 0"/>
-    </joint>
-    <link name="back_caster_wheel_two">
-        <visual>
-            <geometry>
-                <sphere radius="0.014" />
-            </geometry>
-            <material name="red">
-                <color rgba="1 0 0 1"/>
-            </material>
-        </visual>
-        <collision>
-            <geometry>
-                <sphere radius="0.014" />
-            </geometry>
-        </collision>
-        <xacro:inertial_sphere mass="0.1" radius="0.014">
-            <origin xyz="0 0 0" rpy="0 0 0"/>
-        </xacro:inertial_sphere>
-    </link>
-    <gazebo reference="back_caster_wheel_two">
-        <material>Gazebo/Black</material>
-        <mu1>0.005</mu1>
-        <mu2>0.005</mu2>
+        <mu1>0.0001</mu1>
+        <mu2>0.0001</mu2>
     </gazebo>
 </robot>

Commit message: Added joystick control

File: description/robot_core.xacro (robot description, xacro)
@@ -5,4 +5,12 @@
     <!-- BASE LINK -->
     <link name="base_link">
+    </link>
+    <!-- BASE_footprint LINK -->
+    <joint name="base_footprint_joint" type="fixed">
+        <parent link="base_link"/>
+        <child link="base_footprint"/>
+        <origin xyz="0 0 0" rpy="0 0 0"/>
+    </joint>
+    <link name="base_footprint">
     </link>
     <!-- CHASSIS LINK -->

Commit message: fixed color

File: description/robot_core.xacro (robot description, xacro)
@@ -40,5 +40,5 @@
     </link>
     <gazebo reference="chassis">
-        <material>Gazebo/White</material>
+        <material>Gazebo/Orange</material>
     </gazebo>
     <!-- LEFT WHEEL LINK -->
